File: hardware/kicad/Sipeed-M1-v1/Sipeed-M1-v1.kicad_sch (KiCad schematic)
At the start: 89 parts, among them J1 USB_C_, J2 FH34SRJ-24S-0.5SH_50_, Q1 DIS-NMOS, Q2 CHAR-NMOS, SW1 SW_Push, SW2 SW_Push, U1 Sipeed-M1, U11 CH343P, U2 CH343P, U3 ESP32-C3, U4 TPS63070RNMR, U5 MCP23017_SO, U6 BQ29700DSER, U7 USBLC6-2SC6, U8 MCP73871, U9 FE1.1s, Y1 Crystal

Commit message: switched MCU to S3, deleted UART-bridge and usb-hub-IC
Parts:
- removed C15, C16, C20, C3, C38, C39, C4, C40, C41, C43, C48, C5: 100nF, symbol Device:C
- removed C17, C18: 22pF, symbol Device:C
- removed C19: 10uF, symbol Device:C
- removed C21: 1uF, symbol Device:C
- removed FB1, FB4: FerriteBead, symbol Device:FerriteBead_Small
- removed J2: FH34SRJ-24S-0.5SH_50_, FH34SRJ-24S-0.5SH_50_:HRS_FH34SRJ-24S-0.5SH_50_, symbol _M1_symbols:FH34SRJ-24S-0.5SH_50_
- removed Q1: DIS-NMOS, symbol Simulation_SPICE:NMOS
- removed Q2: CHAR-NMOS, symbol Simulation_SPICE:NMOS
- removed R11: 2k, symbol Device:R
- removed R12: 20k, symbol Device:R
- removed R24, R4: 33 O, symbol Device:R
- removed U11, U2: CH343P, Package_DFN_QFN:WCH_QFN-16-1EP_3x3mm_P0.5mm_EP1.8x1.8mm, symbol _M1_symbols:CH343P
- removed U3: ESP32-C3, Package_DFN_QFN:QFN-32-1EP_5x5mm_P0.5mm_EP3.7x3.7mm, symbol _M1_symbols:ESP32-C3
- removed U5: MCP23017_SO, Package_SO:SOIC-28W_7.5x17.9mm_P1.27mm, symbol Interface_Expansion:MCP23017_SO
- removed U9: FE1.1s, Package_SO:SSOP-28_3.9x9.9mm_P0.635mm, symbol Interface_USB:FE1.1s
- removed Y1: Crystal, symbol Device:Crystal
- added J2: JST Connector, symbol MySymbols_ProjectLib:Conn_01x02_Pin
- added J3: Conn_02x20_Odd_Even, symbol Connector_Generic:Conn_02x20_Odd_Even
- added JP1, JP2: Jumper_3_Br, Jumper:SolderJumper-3_P1.3mm_Bridged12_RoundedPad1.0x1.5mm_NumberLabels, symbol Jumper:SolderJumper_3_Bridged123
- added Q2: FS8205A, _M1_FP_lib:FS8205A TSSOP-8_3x3mm_P0.65mm, symbol _M1_symbols:FS8205A
- added SW3, SW4: SW_Push, Button_Switch_THT:SW_PUSH_6mm_H5mm, symbol Switch:SW_Push
- added TP1: TP_PACK-, TestPoint:TestPoint_Pad_D2.0mm, symbol Connector:TestPoint
- added TP2: TP_DOUT, TestPoint:TestPoint_Pad_D2.0mm, symbol Connector:TestPoint
- added TP3: TP_COUT, TestPoint:TestPoint_Pad_D2.0mm, symbol Connector:TestPoint
- added TP4: TP_USB_D-, TestPoint:TestPoint_Pad_D2.0mm, symbol Connector:TestPoint
- added TP5: TP_USB_D+, TestPoint:TestPoint_Pad_D2.0mm, symbol Connector:TestPoint
- added U2: ESP32-S3-WROOM-1U-N8R8, _M1_FP_lib:XCVR_ESP32-S3-WROOM-1U-N8R8, symbol _M1_symbols:ESP32-S3-WROOM-1U-N8R8
- C1, C10, C11, C34, C7: footprint (none) -> Capacitor_SMD:C_0603_1608Metric
- C12, C13, C14, C2, C33, C6, C8, C9: footprint (none) -> Capacitor_SMD:C_1210_3225Metric
- C46: value 100uF -> 100uF 10V Tant; footprint Capacitor_Tantalum_SMD:CP_EIA-3528-12_Kemet-T -> Capacitor_Tantalum_SMD:CP_EIA-6032-28_Kemet-C; symbol Device:C -> Device:C_Polarized
- C47: value 100uF -> 22uF; footprint (none) -> Capacitor_SMD:C_1206_3216Metric
- D1, D2: footprint (none) -> LED_SMD:LED_0603_1608Metric
- F1: value PTC 750mA -> PTC 1.25A
- L2: footprint (none) -> Inductor_SMD:L_6.3x6.3_H3
- R1, R10, R13, R14, R15, R16, R18, R2, R3, R5, R6: footprint (none) -> Resistor_SMD:R_0603_1608Metric
- R11, R12, R7, R8: footprint (none) -> Resistor_SMD:R_0805_2012Metric
- R17: value 10k -> 100 O; footprint (none) -> Resistor_SMD:R_0603_1608Metric
- R19: value 10k -> 100k; footprint (none) -> Resistor_SMD:R_0603_1608Metric
- R20: value 12k -> 100 O; footprint (none) -> Resistor_SMD:R_0603_1608Metric
- R21: value 22 -> 100k; footprint (none) -> Resistor_SMD:R_0603_1608Metric
- R22: value 22 -> 2k; footprint (none) -> Resistor_SMD:R_0603_1608Metric
- R23: value 22 -> 20k; footprint (none) -> Resistor_SMD:R_0603_1608Metric
- R25: value 22 -> 100k; footprint (none) -> Resistor_SMD:R_0805_2012Metric
- R9: value 10kO -> 10k; footprint (none) -> Resistor_SMD:R_0603_1608Metric
- SW1, SW2: footprint (none) -> Button_Switch_THT:SW_PUSH_6mm_H5mm
- TH1: footprint (none) -> Fuse:Fuse_1812_4532Metric
- TP10, TP11, TP13, TP14, TP9: footprint (none) -> TestPoint:TestPoint_Pad_D2.0mm
- TP8: value TP_VBAT -> TP_PACK+; footprint (none) -> TestPoint:TestPoint_Pad_D2.0mm
- U6: footprint BQ29700DSER:SON50P150X150X80-6N -> _M1_FP_lib:BQ29700DSER SON50P150X150X80-6N
Connections:
- net C3D+ is gone; now on net GND: R21.2
- net C3D- is gone; now on an unnamed net: R22.2
- net M1D+ is gone; now on an unnamed net: R23.2
- net VBAT-NEG is gone; now on net CELL-: U6.6 (V-)
- net +3.3V_SYS: now also R3.1, U4.6 (FB2)
- net GND: now also R22.1, R23.1, R25.1, Q2.6, Q2.7, SW3.2, SW4.2, TP1.1; no longer C1.1, R20.1, R3.1, U8.4 (PROG2)
- net VBUS: now also U8.4 (PROG2)
- net at R20.2: now also R21.1, Q2.5
- net at R7.2, R8.2, U4.5 (FB): no longer U4.6 (FB2)
- net FLASH_S3: now reaches R3.2
- net FLASH_S3: now also SW3.1, U2.27 (IO0)
- net RESET_S3: now reaches R18.2
- net RESET_S3: now also C2.1, SW4.1, U2.3 (EN)
- net PACK+: now reaches C1.2
- net PACK+: now also C46.1, C47.1, TP8.1, U6.5 (BAT), U8.14 (V_{BAT}), U8.15 (V_{BAT}), U8.16 (V_{BAT_SENSE}), J2.1 (Pin_1); no longer C2.1
- net CELL-: now reaches R19.2
- net CELL-: now also C1.1, J2.2 (Pin_2), Q2.2, Q2.3
- net at R17.2: now also R19.1, Q2.4
- net C6_P4_PWR_GOOD: no longer names the net of R9.1, U4.2 (PG)
- net CHAR renamed COUT
- net COUT: now also R17.1, TP3.1
- net DISCH renamed DOUT
- net DOUT: now also R20.1, TP2.1
- net FLASH_BTN renamed FLASH_M1
- net M1D- renamed PFM_PWM_SEL
- net PFM_PWM_SEL: now also U4.1 (PS/SYNC), U2.12 (IO8)
- net RESET_BTN renamed RESET_M1
- net RXD-TXM1: no longer names the net of U1.6 (IO5/ISP_Tx)
- net STAT1: no longer names the net of R13.1, U8.8 (STAT1/~{LBO})
- net STAT2: no longer names the net of R14.1, U8.7 (STAT2)
- net TXD-RXM1: no longer names the net of U1.5 (IO4/ISP_Rx)
- net UD+ renamed D+
- net UD- renamed D-
- removed net VBAT: C46.1, C47.1, TP8.1, U4.1 (PS/SYNC), U4.14 (EN), U6.5 (BAT), U8.14 (V_{BAT}), U8.15 (V_{BAT}), U8.16 (V_{BAT_SENSE})
- net VBAT_OUT renamed VSYS
- net VSYS: now also U4.14 (EN)
- removed net VD33O: R17.1, R19.1
- new net: U2.1 (GND), U2.40 (GND), U2.41_1 (GND), U2.41_2 (GND), U2.41_3 (GND), U2.41_4 (GND), U2.41_5 (GND), U2.41_6 (GND), U2.41_7 (GND), U2.41_8 (GND), U2.41_9 (GND)
- new net: Q2.1, Q2.8
- new net RX_BO: JP2.3 (B)
- new net RX_M1: JP2.1 (A)
- new net RX_S3: JP1.2 (C), U2.36 (RXD0)
- new net TX_BO: JP1.3 (B)
- new net TX_M1: JP1.1 (A)
- new net TX_S3: JP2.2 (C), U2.37 (TXD0)
- new net USB_D+: TP5.1, U2.14 (IO20)
- new net USB_D-: TP4.1, U2.13 (IO19)
- no-connect marks 23 -> 3
Other:
- note added: "Buck-Boost-Converter (generates 3.3V for MCUs)"
- note added: "CELL+"
- note added: "CHARGING IC"
- note added: "Connector for LiPo"
- note added: "Flash Button for prog - M1"
- note added: "Flash Button for prog - S3"
- note added: "LOW/Default = PFM, HIGH = PWM-only"
- note added: "MCU - M1"
- note added: "MCU - S3"
- note added: "Reset Button for prog - M1"
- note added: "Reset Button for prog - S3"
- note added: "USB_C Connector"
- note removed: "Buck-Boost-Converter (generates 3.3V for MCUs, switches between USB/LiPo)"
- note removed: "Flash Button for prog"
- note removed: "Reset Button for prog"
- note removed: "USB_C Connector (5V for LiPo loading, DataPins for prog)"
- note removed: "USB_C to UART Bridge IC for M1"
- note removed: "needs physical buttons for flash/reset"
- moved on the sheet: C10, C12, C13, C33, C34, C47, C6, C7, C8, C9, D1, D2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

Commit message: added raspi-scheme breakout and multiple wiring
Parts:
- added C15, C17, C4: 10uF, Capacitor_SMD:C_1210_3225Metric, symbol Device:C
- added C16: 100nF, Capacitor_SMD:C_0603_1608Metric, symbol Device:C
- added C3, C5: 100nF, Capacitor_SMD:C_1210_3225Metric, symbol Device:C
- added D4: D_Schottky, Diode_SMD:D_SOD-123F, symbol Device:D_Schottky
- added JP3, JP4: SJumper, Jumper:SolderJumper-2_P1.3mm_Open_RoundedPad1.0x1.5mm, symbol Jumper:SolderJumper_2_Open
- added JP5: SJ_2_B, Jumper:SolderJumper-2_P1.3mm_Bridged_RoundedPad1.0x1.5mm, symbol Jumper:SolderJumper_2_Bridged
- added R24, R26, R27, R28, R4: 10kO, Resistor_SMD:R_0603_1608Metric, symbol Device:R
- added R29, R30: 4k7, Resistor_SMD:R_0603_1608Metric, symbol Device:R
- added TP6: TP_ID_SD, TestPoint:TestPoint_Pad_D2.0mm, symbol Connector:TestPoint
- added TP7: TP_ID_SC, TestPoint:TestPoint_Pad_D2.0mm, symbol Connector:TestPoint
- F1: footprint (none) -> Fuse:Fuse_1812_4532Metric
- J1: footprint (none) -> Connector_USB:USB_C_Receptacle_HRO_TYPE-C-31-M-12
- J2: footprint (none) -> Connector_JST:JST_PH_S2B-PH-SM4-TB_1x02-1MP_P2.00mm_Horizontal; symbol MySymbols_ProjectLib:Conn_01x02_Pin -> Connector:Conn_01x02_Pin
- J3: footprint (none) -> Connector_PinHeader_2.54mm:PinHeader_2x20_P2.54mm_Vertical
- R10, R6: value 22 O -> 22
- U4: footprint TPS63070RNMR:VREG_TPS63070RNMR -> _M1_FP_lib:VREG_TPS63070RNMR
- renumbered C33 to C18, C34 to C19
Connections:
- net D- is gone; now on net USB_D-: R6.2
- net +3.3V_SYS: now also J3.1 (Pin_1), J3.17 (Pin_17), U2.2 (3V3), C15.1, C16.1, C17.1, C3.1, C4.1, C5.1, R24.1, R26.1, R27.1, R28.1, R29.1, R30.1, R4.1
- net GND: now also J3.20 (Pin_20), J3.25 (Pin_25), J3.30 (Pin_30), J3.34 (Pin_34), J3.39 (Pin_39), J3.6 (Pin_6), J3.9 (Pin_9), C15.2, C16.2, C17.2, C3.2, C4.2, C5.2
- net RX_BO: now also J3.10 (Pin_10)
- net SPI_CS_M1: now also U2.22 (IO14), R4.2
- net SPI_MISO: now also J3.21 (Pin_21), U2.30 (IO37)
- net SPI_MOSI: now also J3.19 (Pin_19), U2.28 (IO35)
- net SPI_SCK: now also J3.23 (Pin_23), U2.29 (IO36)
- net TX_BO: now also J3.8 (Pin_8)
- net USB_D+: now also J1.A6 (D+), J1.B6 (D+), R10.1, U7.3 (I/O2); no longer TP5.1
- net USB_D-: now also J1.A7 (D-), J1.B7 (D-), U7.1 (I/O1); no longer TP4.1
- net VBUS: now also JP5.2 (B)
- net SPI_RST_EPD: now reaches U2.10 (IO17)
- net SPI_BUSY_EPD: now reaches U2.16 (IO46)
- net SPI_CS_BO1: now reaches U2.19 (IO11)
- net SPI_CS_BO1: now also J3.24 (Pin_24), U2.20 (IO12), R26.2, R28.2
- net SPI_CS_BO2: now reaches U2.21 (IO13)
- net SPI_CS_BO2: now also J3.26 (Pin_26), R24.2
- net I2C1_SDA: now reaches U2.4 (IO4)
- net I2C1_SDA: now also J3.3 (Pin_3), JP4.2 (B)
- net I2C1_SCL: now reaches U2.5 (IO5)
- net I2C1_SCL: now also J3.5 (Pin_5), JP3.2 (B)
- net SPI_CS_EPD: now reaches U2.8 (IO15)
- net SPI_CS_EPD: now also R27.2
- net SPI_DC_EPD: now reaches U2.9 (IO16)
- net 5V_HDR: now reaches J3.2 (Pin_2)
- net 5V_HDR: now also J3.4 (Pin_4), D4.1 (K)
- net ID_SD: now reaches J3.27 (Pin_27)
- net ID_SD: now also TP6.1
- net ID_SC: now reaches J3.28 (Pin_28)
- net ID_SC: now also TP7.1
- net CC1: no longer names the net of J1.A5 (CC1), R1.1
- net CC2: no longer names the net of J1.B5 (CC2), R2.1
- net D+: no longer names the net of R10.2
- net D+: now also TP5.1
- new net: D4.2 (A), JP5.1 (A)
- new net: JP3.1 (A), R30.2
- new net: JP4.1 (A), R29.2
- new net: R6.1, TP4.1
- no-connect marks 3 -> 4
Other:
- note added: "INPUT ONLY!"
- note removed: "PIN 7,8,9 SIND BEIM M1W INTERN MIT WIFI BELEGT"
- moved on the sheet: C11, C14, D3, F1, R1, R16, R2, R3, TP10, TP4, TP5, U7

Commit message: added booster for 5v for M1
Parts:
- added C22, C24, C25, C26, C27, C29: 100nF, Capacitor_SMD:C_0603_1608Metric, symbol Device:C
- added C23: 10uF, Capacitor_SMD:C_1206_3216Metric, symbol Device:C
- added C28: 1uF, Capacitor_SMD:C_0805_2012Metric, symbol Device:C
- added C32: 100nF, Capacitor_Tantalum_SMD:CP_EIA-3528-12_Kemet-T, symbol Device:C
- added C49: 10uF, Capacitor_Tantalum_SMD:CP_EIA-3528-12_Kemet-T, symbol Device:C
- added C50: 22uF, Capacitor_Tantalum_SMD:CP_EIA-3528-12_Kemet-T, symbol Device:C
- added D5, D6: D_Schottky, Diode_SMD:D_SOD-123F, symbol Device:D_Schottky
- added IC1: TROPIC01_chip, _M1_FP_lib:QFN-32-1EP_4x4mm_P0.4mm_EP2.65x2.65mm TROPIC01, symbol _M1_symbols:TROPIC01_chip_pub
- added J4: Conn_01x09_Pin, Connector_PinHeader_2.54mm:PinHeader_1x09_P2.54mm_Vertical, symbol Connector:Conn_01x09_Pin
- added J5: Conn_02x03_Odd_Even, Connector_PinSocket_2.54mm:PinSocket_2x03_P2.54mm_Vertical, symbol Connector_Generic:Conn_02x03_Odd_Even
- added JP10: SJ_3_Br12, Jumper:SolderJumper-3_P1.3mm_Bridged12_RoundedPad1.0x1.5mm_NumberLabels, symbol Jumper:SolderJumper_3_Bridged123
- added JP6: Jumper_3_Br, Jumper:SolderJumper-3_P1.3mm_Bridged12_RoundedPad1.0x1.5mm_NumberLabels, symbol Jumper:SolderJumper_3_Bridged123
- added JP7, JP8: Jump_3_Br12, Jumper:SolderJumper-3_P1.3mm_Bridged12_RoundedPad1.0x1.5mm_NumberLabels, symbol Jumper:SolderJumper_3_Bridged123
- added JP9: SJumper, Jumper:SolderJumper-2_P1.3mm_Open_RoundedPad1.0x1.5mm, symbol Jumper:SolderJumper_2_Open
- added L3: 2.2uH, Inductor_SMD:L_6.3x6.3_H3, symbol Device:L
- added R31: 47, Resistor_THT:R_Axial_DIN0207_L6.3mm_D2.5mm_P7.62mm_Horizontal, symbol Device:R
- added R32: 47, Resistor_SMD:R_0603_1608Metric, symbol Device:R
- added R33: 10kO, Resistor_THT:R_Axial_DIN0207_L6.3mm_D2.5mm_P7.62mm_Horizontal, symbol Device:R
- added R34: 100k, Resistor_SMD:R_0603_1608Metric, symbol Device:R
- added R35, R37, R38: 100, Resistor_SMD:R_0603_1608Metric, symbol Device:R
- added R36: 22, Resistor_SMD:R_0603_1608Metric, symbol Device:R
- added R39, R43: 50kO, Resistor_SMD:R_0603_1608Metric, symbol Device:R
- added R40: 47k, Resistor_SMD:R_0603_1608Metric, symbol Device:R
- added R41: 200kO, Resistor_SMD:R_0805_2012Metric, symbol Device:R
- added R42: 370kO, Resistor_SMD:R_0805_2012Metric, symbol Device:R
- added SW5, SW6: SW_Push, Button_Switch_THT:SW_PUSH_6mm_H5mm, symbol Switch:SW_Push
- added TP12: TP_RST_M1, TestPoint:TestPoint_Pad_D2.0mm, symbol Connector:TestPoint
- added TP15: TP_FLASH_M1, TestPoint:TestPoint_Pad_D2.0mm, symbol Connector:TestPoint
- added TP16: TP_RX_M1, TestPoint:TestPoint_Pad_D2.0mm, symbol Connector:TestPoint
- added TP17: TP_TX_M1, TestPoint:TestPoint_Pad_D2.0mm, symbol Connector:TestPoint
- added TP18: TP_ISP_RX_M1, TestPoint:TestPoint_Pad_D2.0mm, symbol Connector:TestPoint
- added TP19: TP_ISP_TX_M1, TestPoint:TestPoint_Pad_D2.0mm, symbol Connector:TestPoint
- added TP20: TP_5V_OUT, TestPoint:TestPoint_Pad_D2.0mm, symbol Connector:TestPoint
- added U3: PAM2401YPADJ, _M1_FP_lib:SON45P300X300X63-13N PAM2401, symbol _M1_symbols:PAM2401YPADJ
- C12, C13, C14, C15, C17, C18, C4, C6, C8, C9: footprint Capacitor_SMD:C_1210_3225Metric -> Capacitor_SMD:C_1206_3216Metric
- C2, C3, C5: footprint Capacitor_SMD:C_1210_3225Metric -> Capacitor_SMD:C_0603_1608Metric
- J2, R30, SW1, SW2, SW3, SW4: now not fitted; now left out of the parts list
- R29: footprint Resistor_SMD:R_0603_1608Metric -> Resistor_THT:R_Axial_DIN0207_L6.3mm_D2.5mm_P7.62mm_Horizontal; now not fitted; now left out of the parts list
- U4: footprint _M1_FP_lib:VREG_TPS63070RNMR -> _M1_FP_lib:TPS63070RNMR
- renumbered C47 to C31
Connections:
- net +3.3V_SYS: now also C23.1, C24.1, C25.1, C26.1, C27.1, C28.1, C29.1, IC1.1 (VCC), IC1.11 (VCC), IC1.22 (PULLUP), IC1.24 (VCC), J4.7 (Pin_7), J5.1 (Pin_1), R33.1, R40.2
- net FLASH_M1: now also TP15.1
- net GND: now also J3.14 (Pin_14), U1.49 (GND), U1.50 (GND), U1.72 (GND), U2.1 (GND), U2.40 (GND), U2.41_1 (GND), U2.41_2 (GND), U2.41_3 (GND), U2.41_4 (GND), U2.41_5 (GND), U2.41_6 (GND), U2.41_7 (GND), U2.41_8 (GND), U2.41_9 (GND), C22.2, C23.2, C24.2, C25.2, C26.2, C27.2, C28.2, C29.2, C32.2, C49.2, C50.2, IC1.10 (PULLDN), IC1.12 (GND), IC1.2 (GND), IC1.23 (GND), IC1.3 (PULLDN), IC1.30 (PULLDN), IC1.31 (PULLDN), IC1.33 (TP), IC1.9 (PULLDN), J4.8 (Pin_8), J5.2 (Pin_2), R34.1, R39.2, R41.1, R43.2, SW5.2, SW6.2, U3.11 (PGND), U3.12 (PGND), U3.13 (EP), U3.6 (AGND)
- net I2C1_SCL: now also JP4.2 (B), U2.4 (IO4), J5.4 (Pin_4); no longer JP3.2 (B), U2.5 (IO5)
- net I2C1_SDA: now also JP3.2 (B), U2.5 (IO5), J5.3 (Pin_3); no longer JP4.2 (B), U2.4 (IO4)
- net RESET_M1: now also C22.1, TP12.1
- net RX_M1: now also U1.42 (IO41), TP16.1
- net SPI_BUSY_EPD: now also J4.1 (Pin_1), JP9.1 (A)
- net SPI_CS_EPD: now also J4.2 (Pin_2)
- net SPI_CS_M1: now also U1.30 (IO29), JP7.3 (B)
- net SPI_DC_EPD: now also J4.3 (Pin_3)
- net SPI_MISO: now also IC1.6 (SDO), J4.9 (Pin_9), JP6.1 (A), R31.1, R32.2; no longer J3.21 (Pin_21), U1.27 (IO26)
- net SPI_MOSI: now also IC1.5 (SDI), J4.5 (Pin_5)
- net SPI_RST_EPD: now also J4.4 (Pin_4)
- net SPI_SCK: now also IC1.7 (SCK), J4.6 (Pin_6), R36.2; no longer U2.29 (IO36)
- net TX_M1: now also U1.41 (IO40), TP17.1
- net VBUS: now also D6.2 (A)
- net VSYS: now also C32.1, C49.1, U3.4 (VIN)
- net PG5V_S3_IO18: now reaches U2.11 (IO18)
- net PG5V_S3_IO18: now also J3.18 (Pin_18)
- net S3_IO3: now reaches U2.15 (IO3)
- net S3_IO3: now also J3.13 (Pin_13)
- net at U2.17 (IO9): now also R37.2
- net S3_IO10: now reaches U2.18 (IO10)
- net S3_IO10: now also J3.11 (Pin_11)
- net S3_IO21: now reaches U2.23 (IO21)
- net S3_IO21: now also IC1.4 (GPO), R34.2, R35.2
- net S3_IO47: now reaches U2.24 (IO47)
- net S3_IO47: now also J3.37 (Pin_37), SW5.1
- net S3_IO48: now reaches U2.25 (IO48)
- net S3_IO48: now also J3.36 (Pin_36), SW6.1
- net S3_IO45: now reaches U2.26 (IO45)
- net S3_IO45: now also J3.15 (Pin_15)
- net I2S_BCLK_IO38: now reaches U2.31 (IO38)
- net I2S_BCLK_IO38: now also J3.12 (Pin_12)
- net I2S_WS_LR_IO39: now reaches U2.32 (IO39)
- net I2S_WS_LR_IO39: now also J3.35 (Pin_35)
- net I2S_DOUT_IO40: now reaches U2.33 (IO40)
- net I2S_DOUT_IO40: now also J3.40 (Pin_40)
- net I2S_DIN_IO41: now reaches U2.34 (IO41)
- net I2S_DIN_IO41: now also J3.38 (Pin_38)
- net S3_IO42: now reaches U2.35 (IO42)
- net S3_IO42: now also J3.16 (Pin_16)
- net PWM0_IO2: now reaches U2.38 (IO2)
- net PWM0_IO2: now also J3.32 (Pin_32)
- net PWM1_IO1: now reaches U2.39 (IO1)
- net PWM1_IO1: now also J3.33 (Pin_33)
- net at U2.6 (IO6): now also R38.2
- net at U2.7 (IO7): now also JP10.2 (C)
- net at J3.22 (Pin_22): now also R35.1
- net S3_IO9: now reaches J3.29 (Pin_29)
- net S3_IO9: now also J5.5 (Pin_5), R37.1
- net S3_IO6: now reaches J3.31 (Pin_31)
- net S3_IO6: now also J5.6 (Pin_6), R38.1
- net GPCLK_IO7: now reaches J3.7 (Pin_7)
- net GPCLK_IO7: now also JP10.3 (B)
- net at U1.5 (IO4/ISP_Rx): now also TP19.1
- net at U1.51 (5V), U1.52 (5V): now also D5.1 (K), D6.1 (K)
- net at U1.6 (IO5/ISP_Tx): now also TP18.1
- net SPI_CS: no longer names the net of U1.26 (IO25)
- removed net SPI_CS_BO1: J3.24 (Pin_24), R26.2, R28.2, U2.19 (IO11), U2.20 (IO12)
- net SPI_CS_BO2 renamed SPI_CS1
- net SPI_CS1: now also JP8.1 (A); no longer J3.26 (Pin_26)
- new net: JP6.3 (B), R31.2
- new net: R36.1, U2.29 (IO36)
- new net: L3.2, U3.1 (LX), U3.2 (LX)
- new net: R42.1, R43.1, U3.7 (FB)
- new net: R41.2, U3.8 (RSET)
- new net: J3.26 (Pin_26), JP8.2 (C)
- new net: J3.21 (Pin_21), JP6.2 (C)
- new net: R32.1, U1.27 (IO26)
- new net: JP9.2 (B), R33.2
- new net: J3.24 (Pin_24), JP7.2 (C)
- new net 5V_BOOST: C50.1, D5.2 (A), R42.2, TP20.1, U3.10 (OUT), U3.9 (OUT)
- new net EN_5V: JP10.1 (A), R39.1, U3.3 (EN)
- new net PG_5V: R40.1, U3.5 (PG)
- new net SPI_CS0: JP7.1 (A), R26.2, U2.20 (IO12)
- new net SPI_CS_TS01: IC1.8 (CSN), JP8.3 (B), R28.2, U2.19 (IO11)
- no-connect marks 4 -> 61
Other:
- note added: "Connector for EPaper"
- note added: "Connector for LiPo (DNP?)"
- note added: "Connector for SAO"
- note added: "Current Limiter"
- note added: "DAMPER-R IF 2x M1 CONNECT!"
- note added: "DIRECT_MISO"
- note added: "EN via S3_IO7"
- note added: "Jumper to M1_onboard, connect one or other, never both!"
- note added: "Jumper to TS01_onboard, connect one or other, never both!"
- note added: "Optional PullUps if needed for Addon!"
- note added: "PACK-"
- note added: "PINS ON CONN - GPIOS ON S3 1 3V3 → +3.3V_SYS 2 5V → from VBUS → Schottky → SJ → 5V_HDR 3 I²C1-SDA → GPIO5 4 5V → same rail as pin 2 5 I²C1-SCL → GPIO4 6 GND 7 FREE /GPCLK → GPIO7 8 UART0-TX → TXD0 (GPIO43) 9 GND 10 UART0-RX → RXD0 (GPIO44) 11 FREE → GPIO10 12 I²S_BCLK → GPIO38 13 FREE /BOOTSTRAP → GPIO3 14 GND 15 FREE /INPUT ONLY /STRAP → GPIO45 16 FREE → GPIO42 17 3V3 → +3.3V_SYS 18 FREE /PG_5V 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"
- note added: "Secure Element - TROPIC01"
- note added: "User Button for Input 1"
- note added: "User Button for Input 2"
- note added: "Voltage Divider sets Output V via ratio"
- note removed: "Connector for LiPo"
- moved on the sheet: C15, C16, C17, C2, C3, C4, C5, D4, J3, JP1, JP2, JP3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

Commit message: added GPIO extender and sorted pcb layout
Parts:
- added C20, C34: 100nF, Capacitor_SMD:C_0603_1608Metric, symbol Device:C
- added C21, C30: 10uF, Capacitor_SMD:C_1206_3216Metric, symbol Device:C
- added D7: D_Schottky, Diode_SMD:D_SOD-123F, symbol Device:D_Schottky
- added JP11: SJ_2_B, Jumper:SolderJumper-2_P1.3mm_Bridged_RoundedPad1.0x1.5mm, symbol Jumper:SolderJumper_2_Bridged
- added JP12, JP13: SJumper, Jumper:SolderJumper-2_P1.3mm_Open_RoundedPad1.0x1.5mm, symbol Jumper:SolderJumper_2_Open
- added R44, R45: 4k7, Resistor_THT:R_Axial_DIN0207_L6.3mm_D2.5mm_P7.62mm_Horizontal, symbol Device:R
- added R46, R47: 10k, Resistor_SMD:R_0603_1608Metric, symbol Device:R
- added SW10, SW11, SW12, SW13, SW14, SW15, SW16, SW7, SW8, SW9: SW_Push, Button_Switch_THT:SW_PUSH_6mm_H5mm, symbol Switch:SW_Push
- added TP21: TP_SDA, symbol Connector:TestPoint
- added TP22: TP_SCK, symbol Connector:TestPoint
- added TP23: TP_INTA, symbol Connector:TestPoint
- added TP24: TP_B6, symbol Connector:TestPoint
- added TP25: TP_B7, symbol Connector:TestPoint
- added TP26: TP_A7, symbol Connector:TestPoint
- added TP27: TP_A6, symbol Connector:TestPoint
- added U5: MCP23017_SO, Package_SO:SOIC-28W_7.5x17.9mm_P1.27mm, symbol Interface_Expansion:MCP23017_SO
- JP3, JP4: footprint Jumper:SolderJumper-2_P1.3mm_Open_RoundedPad1.0x1.5mm -> Jumper:SolderJumper-2_P1.3mm_Bridged_RoundedPad1.0x1.5mm
- R29: footprint Resistor_THT:R_Axial_DIN0207_L6.3mm_D2.5mm_P7.62mm_Horizontal -> Resistor_SMD:R_0603_1608Metric; now fitted; now in the parts list
- R30: now fitted; now in the parts list
Connections:
- net +3.3V_SYS: now also C34.2, R44.1, R45.1, R46.1, R47.1, U5.9 (VDD)
- net 5V_BOOST: now also JP11.2 (B)
- net 5V_HDR: now also C20.1, C21.1, C30.1, D7.1 (K)
- net GND: now also C20.2, C21.2, C30.2, C34.1, SW10.2, SW11.2, SW12.2, SW13.2, SW14.2, SW15.2, SW16.2, SW7.2, SW8.2, SW9.2, U5.10 (VSS), U5.15 (A0), U5.16 (A1), U5.17 (A2)
- net I2C1_SCL: now also JP13.2 (B), TP22.1, U5.12 (SCK)
- net I2C1_SDA: now also JP12.2 (B), TP21.1, U5.13 (SDA)
- net S3_IO47: no longer SW5.1
- net S3_IO48: now also R47.2, TP23.1, U5.20 (INTA); no longer SW6.1
- net VSYS: now also L3.1
- new net: JP13.1 (A), R45.2
- new net: TP26.1, U5.28 (GPA7)
- new net: TP25.1, U5.8 (GPB7)
- new net: D7.2 (A), JP11.1 (A)
- new net: R46.2, U5.18 (~{RESET})
- new net: TP24.1, U5.7 (GPB6)
- new net: TP27.1, U5.27 (GPA6)
- new net: JP12.1 (A), R44.2
- new net BTN_0: SW5.1, U5.1 (GPB0)
- new net BTN_1: SW6.1, U5.2 (GPB1)
- new net BTN_2: SW7.1, U5.3 (GPB2)
- new net BTN_3: SW8.1, U5.4 (GPB3)
- new net BTN_4: SW9.1, U5.5 (GPB4)
- new net BTN_5: SW10.1, U5.6 (GPB5)
- new net BTN_6: SW11.1, U5.21 (GPA0)
- new net BTN_7: SW12.1, U5.22 (GPA1)
- new net BTN_8: SW13.1, U5.23 (GPA2)
- new net BTN_9: SW14.1, U5.24 (GPA3)
- new net BTN_NO: SW16.1, U5.26 (GPA5)
- new net BTN_YES: SW15.1, U5.25 (GPA4)
- no-connect marks 61 -> 62
Other:
- note added: "5V Boost Converter"
- note added: "GPIO Expander"
- note added: "User Buttons 0-9 YES NO"
- note removed: "User Button for Input 1"
- note removed: "User Button for Input 2"
- moved on the sheet: C1, C11, C12, C13, C14, C22, C25, C26, C27, C28, C31, C32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

Commit message: added schem changes
Parts:
- TP21, TP22, TP23, TP24, TP25, TP26, TP27: footprint (none) -> TestPoint:TestPoint_Pad_D2.0mm
Changed lines of the file:
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@@
 			)
 		)
-		(property "Footprint" ""
+		(property "Footprint" "TestPoint:TestPoint_Pad_D2.0mm"
 			(at 232.41 240.03 0)
 			(effects
@@
 			)
 		)
-		(property "Footprint" ""
+		(property "Footprint" "TestPoint:TestPoint_Pad_D2.0mm"
 			(at 232.41 217.17 0)
 			(effects
@@
 			)
 		)
-		(property "Footprint" ""
+		(property "Footprint" "TestPoint:TestPoint_Pad_D2.0mm"
 			(at 232.41 214.63 0)
 			(effects
@@
 			)
 		)
-		(property "Footprint" ""
+		(property "Footprint" "TestPoint:TestPoint_Pad_D2.0mm"
 			(at 199.39 196.85 0)
 			(effects
@@
 			)
 		)
-		(property "Footprint" ""
+		(property "Footprint" "TestPoint:TestPoint_Pad_D2.0mm"
 			(at 232.41 237.49 0)
 			(effects
@@
 			)
 		)
-		(property "Footprint" ""
+		(property "Footprint" "TestPoint:TestPoint_Pad_D2.0mm"
 			(at 199.39 203.2 0)
 			(effects
@@
 			)
 		)
-		(property "Footprint" ""
+		(property "Footprint" "TestPoint:TestPoint_Pad_D2.0mm"
 			(at 190.5 217.17 0)
 			(effects
