File: cdc-badge/cdc-badge.kicad_sch (KiCad schematic)
At the start: 134 parts, among them J1 USB_C, J2 JST S2B-PH-SM4-TB, J3 Conn_02x20_Odd_Even, J4 Conn_Grove, J5 Conn_02x03_Odd_Even, J6 Conn_01x06, J7 Conn_01x24, Q1 Si1308EDL, Q2 SS8050, SW0 0, SW1 1, SW10 YES, SW11 NO, SW12 power on/reset, SW13 reset, SW14 flash/power off, SW15 MST-22D18G2 3J, SW16 MST-22D18G2 3J, SW2 2, SW3 3, SW4 4, SW5 5, SW6 6, SW7 7, SW8 8, SW9 9, U1 ESP32-S3-WROOM-1-N16R8, U2 TCA9535PWR, U3 TROPIC01, U4 TPS613222ADBV, U6 BQ25895RTW, U7 USBLC6-2SC6, U8 TLV62569DBV

Commit message: schematic: ceetee reviews, secure element
Add 0 ohm resistor to ease power glitch testing.
Add pads for pull up on GPO/IRQ, and pull down on CS.
Parts:
- added R36, R37: 47k, Resistor_SMD:R_0603_1608Metric, symbol Device:R_Small
- added R41: 0, Resistor_SMD:R_0603_1608Metric, symbol Device:R_Small
Connections:
- net +3.3V: now also R41.2; no longer C2.1, C3.1, C4.1, R3.1, U3.1 (VCC), U3.11 (VCC), U3.22 (PULLUP), U3.24 (VCC)
- net GND: now also R36.2
- net SPI_CS_TR01: now also R37.2
- net TR01_IRQ: now also R36.1
- new net: C2.1, C3.1, C4.1, R3.1, R37.1, R41.1, U3.1 (VCC), U3.11 (VCC), U3.22 (PULLUP), U3.24 (VCC)
Other:
- note added: "take out for power glitching"
- moved on the sheet: C2, C3, C4, R3, U3
